Commit message: Updated LMX11 orientation, host, and added frame_id

File: urdf/sick_lms1xx.urdf.xacro (robot description, xacro)
@@ -36,5 +36,5 @@
       </inertial>
       <visual>
-        <origin xyz="0 0 0" rpy="0 0 0" />
+        <origin xyz="0 0 0" rpy="${-M_PI} 0 0" />
         <geometry>
           <!-- Origin of this mesh is the focal point of the LIDAR. -->
@@ -43,5 +43,5 @@
       </visual>
       <collision>
-        <origin xyz="0 0 -0.05" rpy="0 0 0" />
+        <origin xyz="0 0 -0.05" rpy="${-M_PI} 0 0" />
         <geometry>
           <box size="0.105 0.1 0.1" />

Commit message: Fixed lidar orientation

File: urdf/sick_lms1xx.urdf.xacro (robot description, xacro)
@@ -36,5 +36,5 @@
       </inertial>
       <visual>
-        <origin xyz="0 0 0" rpy="${-M_PI} 0 0" />
+        <origin xyz="0 0 0" rpy="0 0 0" />
         <geometry>
           <!-- Origin of this mesh is the focal point of the LIDAR. -->
@@ -43,5 +43,5 @@
       </visual>
       <collision>
-        <origin xyz="0 0 -0.05" rpy="${-M_PI} 0 0" />
+        <origin xyz="0 0 -0.05" rpy="0 0 0" />
         <geometry>
           <box size="0.105 0.1 0.1" />
